Commit message: Corrected mjcf and urdf file using relative coordinates and original measurements; need to update measurements and collision and COM

File: resources/robots/STEP_6_DOF/urdf/STEP-6-DOF.urdf (robot description, URDF)
Before this commit: robot STEP_6_dof, 9 links, 8 joints
Links:
- removed link base_link
- added link base; collision mesh filename=../meshes/link00.stl scale=0.001 0.001 0.001; visual mesh filename=../meshes/link00.stl scale=0.001 0.001 0.001
- link left_ankle_pitch_link: geometry collision mesh filename=../meshes/link4.stl scale=0.001 0.001 0.001; visual mesh filename=../meshes/link4.stl scale=0.001 0.001 0.001
- link left_hip_pitch_link: geometry collision mesh filename=../meshes/link2.stl scale=0.001 0.001 0.001; visual mesh filename=../meshes/link2.stl scale=0.001 0.001 0.001
- link left_hip_roll_link: geometry collision mesh filename=../meshes/link1.stl scale=0.001 0.001 0.001; visual mesh filename=../meshes/link1.stl scale=0.001 0.001 0.001
- link left_knee_pitch_link: geometry collision mesh filename=../meshes/link3.stl scale=0.001 0.001 0.001; visual mesh filename=../meshes/link3.stl scale=0.001 0.001 0.001
- link right_ankle_pitch_link: geometry collision mesh filename=../meshes/link4_m.stl scale=0.001 0.001 0.001; visual mesh filename=../meshes/link4_m.stl scale=0.001 0.001 0.001
- link right_hip_pitch_link: geometry collision mesh filename=../meshes/link2_m.stl scale=0.001 0.001 0.001; visual mesh filename=../meshes/link2_m.stl scale=0.001 0.001 0.001
- link right_hip_roll_link: geometry collision mesh filename=../meshes/link1_m.stl scale=0.001 0.001 0.001; visual mesh filename=../meshes/link1_m.stl scale=0.001 0.001 0.001
- link right_knee_pitch_link: geometry collision mesh filename=../meshes/link3_m.stl scale=0.001 0.001 0.001; visual mesh filename=../meshes/link3_m.stl scale=0.001 0.001 0.001
Joints:
- joint left_ankle_pitch: limit lower=-0.23 upper=0.23 effort=8 velocity=10 -> lower=-0.23 upper=0.23 effort=10 velocity=10; origin xyz=-0.082 0.05 -0.535 -> xyz=-0.012 0.0 -0.265 rpy=0 0 0
- joint left_hip_pitch: limit lower=-0.93 upper=0.93 effort=8 velocity=10 -> lower=-0.93 upper=0.93 effort=10 velocity=10; origin xyz=-0.08 0.05 0.0 -> xyz=0.01 0.05 0.0 rpy=0 0 0
- joint left_hip_roll: limit lower=-0.05 upper=0.05 effort=8 velocity=10 -> lower=-0.05 upper=0.05 effort=10 velocity=10; origin xyz=-0.09 0 0 -> xyz=-0.09 0 0 rpy=0 0 0; parent base_link -> base
- joint left_knee_pitch: limit lower=-0.93 upper=0.93 effort=8 velocity=10 -> lower=-0.93 upper=0.93 effort=10 velocity=10; origin xyz=-0.07 0.05 -0.27 -> xyz=0.01 0.0 -0.27 rpy=0 0 0
- joint right_ankle_pitch: limit lower=-0.23 upper=0.23 effort=8 velocity=10 -> lower=-0.23 upper=0.23 effort=10 velocity=10; origin xyz=-0.082 0.05 -0.535 -> xyz=0.012 0.0 -0.265 rpy=0 0 0
- joint right_hip_pitch: limit lower=-0.93 upper=0.93 effort=8 velocity=10 -> lower=-0.93 upper=0.93 effort=10 velocity=10; origin xyz=0.08 0.05 0.0 -> xyz=-0.01 0.05 0.0 rpy=0 0 0
- joint right_hip_roll: limit lower=-0.05 upper=0.05 effort=8 velocity=10 -> lower=-0.05 upper=0.05 effort=10 velocity=10; origin xyz=0.09 0 0 -> xyz=0.09 0 0 rpy=0 0 0; parent base_link -> base
- joint right_knee_pitch: limit lower=-0.93 upper=0.93 effort=8 velocity=10 -> lower=-0.93 upper=0.93 effort=10 velocity=10; origin xyz=0.07 0.05 -0.27 -> xyz=-0.01 0.0 -0.27 rpy=0 0 0

Commit message: urdf file is changed to face x positive direction rather than y axis direction

File: resources/robots/STEP_6_DOF/urdf/STEP-6-DOF.urdf (robot description, URDF)
Before this commit: robot STEP_6_dof, 9 links, 8 joints
Joints:
- joint left_ankle_pitch: axis 1 0 0 -> 0 1 0; origin xyz=-0.012 0.0 -0.265 rpy=0 0 0 -> xyz=0.0 0.012 -0.265 rpy=0 0 0
- joint left_hip_pitch: axis 1 0 0 -> 0 1 0; origin xyz=0.01 0.05 0.0 rpy=0 0 0 -> xyz=0.05 -0.01 0.0 rpy=0 0 0
- joint left_hip_roll: axis 0 1 0 -> 1 0 0; origin xyz=-0.09 0 0 rpy=0 0 0 -> xyz=0 0.09 0 rpy=0 0 0
- joint left_knee_pitch: axis 1 0 0 -> 0 1 0; origin xyz=0.01 0.0 -0.27 rpy=0 0 0 -> xyz=0.0 -0.01 -0.27 rpy=0 0 0
- joint right_ankle_pitch: axis 1 0 0 -> 0 1 0; origin xyz=0.012 0.0 -0.265 rpy=0 0 0 -> xyz=0.0 -0.012 -0.265 rpy=0 0 0
- joint right_hip_pitch: axis 1 0 0 -> 0 1 0; origin xyz=-0.01 0.05 0.0 rpy=0 0 0 -> xyz=0.05 0.01 0.0 rpy=0 0 0
- joint right_hip_roll: axis 0 1 0 -> 1 0 0; origin xyz=0.09 0 0 rpy=0 0 0 -> xyz=0 -0.09 0 rpy=0 0 0
- joint right_knee_pitch: axis 1 0 0 -> 0 1 0; origin xyz=-0.01 0.0 -0.27 rpy=0 0 0 -> xyz=0.0 0.01 -0.27 rpy=0 0 0

Commit message: simplified collision to avoid unnecessary collision during training

File: resources/robots/STEP_6_DOF/urdf/STEP-6-DOF.urdf (robot description, URDF)
Before this commit: robot STEP_6_dof, 9 links, 8 joints
Links:
- link base: geometry collision box size=0.1 0.1 0.1; visual mesh filename=../meshes/link00.stl scale=0.001 0.001 0.001
- link left_hip_roll_link: geometry visual mesh filename=../meshes/link1.stl scale=0.001 0.001 0.001
- link left_knee_pitch_link: geometry visual mesh filename=../meshes/link3.stl scale=0.001 0.001 0.001
- link right_hip_roll_link: geometry visual mesh filename=../meshes/link1_m.stl scale=0.001 0.001 0.001
- link right_knee_pitch_link: geometry visual mesh filename=../meshes/link3_m.stl scale=0.001 0.001 0.001
Joints:
- joint left_hip_roll: limit lower=-0.05 upper=0.05 effort=10 velocity=10 -> lower=-0.15 upper=0.15 effort=10 velocity=10
- joint right_hip_roll: limit lower=-0.05 upper=0.05 effort=10 velocity=10 -> lower=-0.15 upper=0.15 effort=10 velocity=10

Commit message: added placeholders for inertia tensors

File: resources/robots/STEP_6_DOF/urdf/STEP-6-DOF.urdf (robot description, URDF)
Before this commit: robot STEP_6_dof, 9 links, 8 joints
Links:
- link base: mass None -> 0.5
- link left_ankle_pitch_link: mass None -> 0.1
- link left_hip_pitch_link: mass None -> 0.2
- link left_hip_roll_link: mass None -> 0.1
- link left_knee_pitch_link: mass None -> 0.2
- link right_ankle_pitch_link: mass None -> 0.1
- link right_hip_pitch_link: mass None -> 0.2
- link right_hip_roll_link: mass None -> 0.1
- link right_knee_pitch_link: mass None -> 0.2

Commit message: updated urdf file

File: resources/robots/STEP_6_DOF/urdf/STEP-6-DOF.urdf (robot description, URDF)
Before this commit: robot STEP_6_dof, 9 links, 8 joints
Links:
- link base: geometry collision box size=0.1 0.1 0.1; visual mesh filename=../meshes/base_link.stl scale=0.001 0.001 0.001
- link left_ankle_pitch_link: mass 0.1 -> 0.16; geometry collision box size=0.07 0.01 0.12; visual mesh filename=../meshes/left_ankle_pitch_link.stl scale=0.001 0.001 0.001
- link left_hip_pitch_link: mass 0.2 -> 0.3; geometry collision mesh filename=../meshes/left_hip_pitch_link.stl scale=0.001 0.001 0.001; visual mesh filename=../meshes/left_hip_pitch_link.stl scale=0.001 0.001 0.001
- link left_hip_roll_link: mass 0.1 -> 0.24; geometry collision mesh filename=../meshes/left_hip_roll_link.stl scale=0.001 0.001 0.001; visual mesh filename=../meshes/left_hip_roll_link.stl scale=0.001 0.001 0.001
- link left_knee_pitch_link: geometry collision mesh filename=../meshes/left_knee_pitch_link.stl scale=0.001 0.001 0.001; visual mesh filename=../meshes/left_knee_pitch_link.stl scale=0.001 0.001 0.001
- link right_ankle_pitch_link: mass 0.1 -> 0.16; geometry collision box size=0.07 0.01 0.12; visual mesh filename=../meshes/right_ankle_pitch_link.stl scale=0.001 0.001 0.001
- link right_hip_pitch_link: mass 0.2 -> 0.3; geometry collision mesh filename=../meshes/right_hip_pitch_link.stl scale=0.001 0.001 0.001; visual mesh filename=../meshes/right_hip_pitch_link.stl scale=0.001 0.001 0.001
- link right_hip_roll_link: mass 0.1 -> 0.24; geometry collision mesh filename=../meshes/right_hip_roll_link.stl scale=0.001 0.001 0.001; visual mesh filename=../meshes/right_hip_roll_link.stl scale=0.001 0.001 0.001
- link right_knee_pitch_link: geometry collision mesh filename=../meshes/right_knee_pitch_link.stl scale=0.001 0.001 0.001; visual mesh filename=../meshes/right_knee_pitch_link.stl scale=0.001 0.001 0.001
