Commit message: Fixed the NaN issue by reducing mass randomization; Created simplified URDF for STEP-8-DOF

File: resources/robots/STEP_8_DOF/urdf/STEP-8-DOF.urdf (robot description, URDF)
Before this commit: robot onshape, 19 links, 18 joints
Links:
- removed link back_hip_link
- removed link base
- removed link depth_camera
- removed link front_hip_link
- removed link left_hip_pitch_motor
- removed link left_hip_roll_motor
- removed link left_hip_roll_to_pitch_link
- removed link left_knee_motor
- removed link left_thigh_link
- removed link right_hip_pitch_motor
- removed link right_hip_roll_motor
- removed link right_hip_roll_to_pitch_link
- removed link right_knee_motor
- removed link right_thigh_link
- added link assembled_base, mass 1.2750789266545348166; collision box size=0.2 0.1 0.1; visual mesh filename=../meshes/assembled_base.stl
- added link left_hip_roll_assembled_link, mass 0.53489494813292881581; collision mesh filename=../meshes/left_hip_roll_assembled_link.stl; visual mesh filename=../meshes/left_hip_roll_assembled_link.stl
- added link left_thigh_assembled_link, mass 0.38042477577232980401; collision mesh filename=../meshes/left_thigh_assembled_link.stl; visual mesh filename=../meshes/left_thigh_assembled_link.stl
- added link right_hip_roll_assembled_link, mass 0.53488105014710862761; collision mesh filename=../meshes/right_hip_roll_assembled_link.stl; visual mesh filename=../meshes/right_hip_roll_assembled_link.stl
- added link right_thigh_assembled_link, mass 0.38042405171223231397; collision mesh filename=../meshes/right_thigh_assembled_link.stl; visual mesh filename=../meshes/right_thigh_assembled_link.stl
- link additional_weight: mass 0.77795469648269044427 -> 0.79579314812178392202
- link left_foot: mass 0.14503328477819069087 -> 0.14503328474795140757
- link left_shin: mass 0.18385415303260232989 -> 0.18385415329439017129
- link right_foot: mass 0.14503328477818819287 -> 0.14503328477161642196
- link right_shin: mass 0.18385415257934586974 -> 0.18385415284334488684
Joints:
- removed joint additional_weight_to_base_fixed_joint
- removed joint back_linkage_to_left_hip_roll_motor_fixed_joint
- removed joint depth_camera_to_base_fixed_joint
- removed joint front_linkage_to_base_fixed_joint
- removed joint left_hip_pitch_motor_to_linkage_fixed_joint
- removed joint left_hip_roll_motor_to_front_linkage_fixed_joint
- removed joint left_knee_motor_to_thigh_fixed_joint
- removed joint right_hip_pitch_motor_to_linkage_fixed_joint
- removed joint right_hip_roll_motor_to_front_linkage_fixed_joint
- removed joint right_knee_motor_to_thigh_fixed_joint
- added joint additional_weight_joint: type fixed, parent assembled_base, child additional_weight, origin xyz=0.0017373457116546199477 4.8047933443529507216e-06 0.60299999999999998046 rpy=-3.141592653589793116 -1.6568748037485875154e-19 -2.0219008759515637583e-35, axis 0 0 1, limit effort=40 velocity=7
- joint left_ankle_joint: limit lower=-0.52359877559829881566 upper=0.52359877559829881566 effort=8 velocity=22 -> lower=-0.52359877559829881566 upper=0.52359877559829881566 effort=40 velocity=7; origin xyz=-0.0032963899599866078316 0.26680321649979088505 0.013000000000000698497 rpy=-4.2351647362715026357e-22 2.957703526540456096e-16 -1.0927227567586433637e-12 -> xyz=-0.0032963899599866147705 0.26680321649979094056 0.012956114963095885506 rpy=3.6779187009318430813e-16 2.7346502719546166981e-16 -3.8824481999271071847e-12
- joint left_hip_pitch_joint: child left_thigh_link -> left_thigh_assembled_link; limit lower=-1.570796326794896558 upper=0.34906585039886589561 effort=8 velocity=22 -> lower=-1.570796326794896558 upper=0.34906585039886589561 effort=40 velocity=7; origin xyz=0.018003009044958225016 0.031175177069699022692 -0.033000000000000195843 rpy=-9.5291206566108472172e-21 -3.5561831257524570087e-17 1.6575893780495051809e-12 -> xyz=-0.020714482720959506712 -1.2195219323100914277e-06 -0.056302758297119864794 rpy=-3.1415746391819041605 1.5707963265842519451 0; parent left_hip_pitch_motor -> left_hip_roll_assembled_link
- joint left_hip_roll_joint: child left_hip_roll_to_pitch_link -> left_hip_roll_assembled_link; limit lower=-0.26179938779914940783 upper=0.26179938779914940783 effort=8 velocity=22 -> lower=-0.26179938779914940783 upper=0.26179938779914940783 effort=40 velocity=7; origin xyz=0.0011510892776742560895 0.032979918033173183378 0.0040000000000000660028 rpy=-3.141592653589793116 3.0791341698589194905e-17 -1.1290875491096140677e-06 -> xyz=-0.041193597110977836495 0.089887544641074693108 -0.018310449527667391895 rpy=1.570796326794896558 -8.3266726846886681367e-16 -1.5680307395761954314; parent left_hip_roll_motor -> assembled_base
- joint left_knee_joint: limit lower=0 upper=0.87266462599716476678 effort=8 velocity=22 -> lower=0 upper=0.87266462599716476678 effort=40 velocity=7; origin xyz=3.2816069428266703145e-06 -0.033999999841633168907 0.0040000000000004103454 rpy=3.1415926535897891192 -3.3827107781547738341e-17 -6.1823809722771156113e-13 -> xyz=-1.1791795445987435231e-05 0.26696937369610784785 -0.0055469999999987473771 rpy=1.2243691845971463006e-16 6.0211425091664846854e-17 2.8257782194518543241e-21; parent left_knee_motor -> left_thigh_assembled_link
- joint right_ankle_joint: limit lower=-0.52359877559829881566 upper=0.52359877559829881566 effort=8 velocity=22 -> lower=-0.52359877559829881566 upper=0.52359877559829881566 effort=40 velocity=7; origin xyz=0.0033478924446542525362 -0.26680257520792788339 0.013000000000000044506 rpy=3.141592653589793116 -2.8406096919120211241e-16 -8.250218779494172183e-19 -> xyz=0.0033478924446542577403 -0.26680257520792799442 0.01295611496309617694 rpy=3.141592653589793116 -2.7996088473986045116e-16 -2.0021163556764444259e-24
- joint right_hip_pitch_joint: child right_thigh_link -> right_thigh_assembled_link; limit lower=-0.34906585039886589561 upper=1.570796326794896558 effort=8 velocity=22 -> lower=-0.34906585039886589561 upper=1.570796326794896558 effort=40 velocity=7; origin xyz=-0.017996990787359258557 -0.031178651712344906954 -0.033000000000000286049 rpy=9.2382707183473101761e-18 1.4745149545802783265e-17 1.1926713100003838507e-07 -> xyz=0.020714482720954302541 1.219252338362231125e-06 -0.056297241554987526024 rpy=1.8014408059877152129e-05 1.5707963267916837946 0; parent right_hip_pitch_motor -> right_hip_roll_assembled_link
- joint right_hip_roll_joint: child right_hip_roll_to_pitch_link -> right_hip_roll_assembled_link; limit lower=-0.26179938779914940783 upper=0.26179938779914940783 effort=8 velocity=22 -> lower=-0.26179938779914940783 upper=0.26179938779914940783 effort=40 velocity=7; origin xyz=0.001151089277675657746 0.0329799180331730446 0.0039999999999999619194 rpy=3.1415926535897917837 1.6913553890773881496e-17 1.0824674490095284158e-15 -> xyz=-0.040695792046267699471 -0.090111766967618897595 -0.018307206934415617278 rpy=1.570796326794896558 9.7189651803362053343e-16 -1.5680307395761954314; parent right_hip_roll_motor -> assembled_base
- joint right_knee_joint: limit lower=-0.87266462599716476678 upper=0 effort=8 velocity=22 -> lower=-0.87266462599716476678 upper=0 effort=40 velocity=7; origin xyz=3.2816069418274695924e-06 0.033999999841633807285 0.0039999999999997051803 rpy=-3.1415926535897895633 -3.426078865054340074e-17 7.0324984147583861797e-16 -> xyz=6.3326415581058115301e-05 -0.26696936644585766985 -0.0055469999999988583994 rpy=6.9117888495950917298e-19 -2.1487086728401866803e-17 2.3825871257081570997e-24; parent right_knee_motor -> right_thigh_assembled_link

Commit message: Updated and fixed the joints' rotation directions in the urdf file

File: resources/robots/STEP_8_DOF/urdf/STEP-8-DOF.urdf (robot description, URDF)
Before this commit: robot onshape, 10 links, 9 joints
Links:
- link assembled_base: mass 1.2750789266545348166 -> 1.2750789266545345946
- link left_shin: mass 0.18385415329439017129 -> 0.18385415329439019905
- link left_thigh_assembled_link: mass 0.38042477577232980401 -> 0.3804247757723297485
- link right_foot: mass 0.14503328477161642196 -> 0.14503328477161644972
- link right_hip_roll_assembled_link: mass 0.53488105014710862761 -> 0.53488105014710873863
- link right_shin: mass 0.18385415284334488684 -> 0.18385415284334485908
- link right_thigh_assembled_link: mass 0.38042405171223231397 -> 0.38042405171223225846
Joints:
- joint left_ankle_joint: origin xyz=-0.0032963899599866147705 0.26680321649979094056 0.012956114963095885506 rpy=3.6779187009318430813e-16 2.7346502719546166981e-16 -3.8824481999271071847e-12 -> xyz=-0.0032963899599866147705 -0.26680321649979094056 -0.012956114963095885506 rpy=-3.1415926535897926719 -2.7346502719546166981e-16 3.8824481999271071847e-12
- joint left_knee_joint: limit lower=0 upper=0.87266462599716476678 effort=40 velocity=7 -> lower=-0.87266462599716476678 upper=-0 effort=40 velocity=7; origin xyz=-1.1791795445987435231e-05 0.26696937369610784785 -0.0055469999999987473771 rpy=1.2243691845971463006e-16 6.0211425091664846854e-17 2.8257782194518543241e-21 -> xyz=-1.1791795445987435231e-05 0.26696937369610784785 -0.0055469999999987473771 rpy=-3.141592653589793116 6.0211425091664846854e-17 2.8257782194518543241e-21
- joint right_ankle_joint: origin xyz=0.0033478924446542577403 -0.26680257520792799442 0.01295611496309617694 rpy=3.141592653589793116 -2.7996088473986045116e-16 -2.0021163556764444259e-24 -> xyz=0.0033478924446542577403 0.26680257520792799442 -0.01295611496309617694 rpy=3.141592653589793116 2.7996088473986045116e-16 2.0021163556764444259e-24
- joint right_knee_joint: limit lower=-0.87266462599716476678 upper=0 effort=40 velocity=7 -> lower=-0 upper=0.87266462599716476678 effort=40 velocity=7; origin xyz=6.3326415581058115301e-05 -0.26696936644585766985 -0.0055469999999988583994 rpy=6.9117888495950917298e-19 -2.1487086728401866803e-17 2.3825871257081570997e-24 -> xyz=6.3326415581058115301e-05 -0.26696936644585766985 -0.0055469999999988583994 rpy=-3.141592653589793116 -2.1487086728401866803e-17 2.3825871257081570997e-24
