Commit message: New urdf for 10 DOF

File: resources/robots/STEP_10_DOF/urdf/STEP-10-DOF.urdf (robot description, URDF)
Before this commit: robot onshape, 12 links, 11 joints
Links:
- removed link left_foot
- removed link left_shin
- removed link left_thigh_assembled_link
- removed link right_foot
- removed link right_shin
- removed link right_thigh_assembled_link
- added link left_ankle_motor, mass 0.4377081912156142729; collision mesh filename=../meshes/left_ankle_motor.stl; visual mesh filename=../meshes/left_ankle_motor.stl
- added link left_foot_10_dof_link, mass 0.17789809743893272853; collision mesh filename=../meshes/left_foot_10_dof_link.stl; visual mesh filename=../meshes/left_foot_10_dof_link.stl
- added link left_knee_motor, mass 0.43770819121562731802; collision mesh filename=../meshes/left_knee_motor.stl; visual mesh filename=../meshes/left_knee_motor.stl
- added link left_shin_motor_down_link, mass 0.24065665756599849412; collision mesh filename=../meshes/left_shin_motor_down_link.stl; visual mesh filename=../meshes/left_shin_motor_down_link.stl
- added link left_thigh_link, mass 0.24065665756599849412; collision mesh filename=../meshes/left_thigh_link.stl; visual mesh filename=../meshes/left_thigh_link.stl
- added link right_ankle_motor, mass 0.4377081912156142729; collision mesh filename=../meshes/right_ankle_motor.stl; visual mesh filename=../meshes/right_ankle_motor.stl
- added link right_foot_10_dof_link, mass 0.1778975924553742316; collision mesh filename=../meshes/right_foot_10_dof_link.stl; visual mesh filename=../meshes/right_foot_10_dof_link.stl
- added link right_knee_motor, mass 0.43770819121563186993; collision mesh filename=../meshes/right_knee_motor.stl; visual mesh filename=../meshes/right_knee_motor.stl
- added link right_shin_motor_down_link, mass 0.24065546894893422025; collision mesh filename=../meshes/right_shin_motor_down_link.stl; visual mesh filename=../meshes/right_shin_motor_down_link.stl
- added link right_thigh_link, mass 0.24065546894893422025; collision mesh filename=../meshes/right_thigh_link.stl; visual mesh filename=../meshes/right_thigh_link.stl
- link 10_dof_base_link: mass 1.1682801127211333014 -> 1.2245306366669659326; geometry collision box size=0.2 0.1 0.1; visual mesh filename=../meshes/torso.stl
- link left_hip_roll_assembled_link: mass 0.53489494813292903785 -> 0.23040104617725792879; geometry collision mesh filename=../meshes/left_hip_roll_assembled_link.stl; visual mesh filename=../meshes/left_hip_roll_assembled_link.stl
- link left_hip_yaw_assembled_link: mass 0.53489494813292881581 -> 0.23040104617725787328
- link right_hip_roll_assembled_link: mass 0.53488105014710873863 -> 0.23039505974855084558; geometry collision mesh filename=../meshes/right_hip_roll_assembled_link.stl; visual mesh filename=../meshes/right_hip_roll_assembled_link.stl
- link right_hip_yaw_assembled_link: mass 0.53488105014710873863 -> 0.23039505974855084558
Joints:
- added joint left_ankle_motor_to_shin: type fixed, parent left_shin_motor_down_link, child left_ankle_motor, origin xyz=8.2040104280228787204e-05 -0.23294457981559668625 0.0015469999999988409689 rpy=6.2242860876268239146e-15 -2.5280088545069896347e-17 2.6624875966549861968e-24, axis 0 0 1, limit effort=8 velocity=12
- added joint left_knee_motor_to_thigh: type fixed, parent left_thigh_link, child left_knee_motor, origin xyz=8.2040104280235726097e-05 0.23294457981559649196 -0.0015469999999995209805 rpy=-3.1415926535897900074 2.4644137901954597791e-17 -6.6174449004242228683e-24, axis 0 0 1, limit effort=8 velocity=12
- added joint right_ankle_motor_to_shin: type fixed, parent right_shin_motor_down_link, child right_ankle_motor, origin xyz=-3.7073482355147457934e-05 0.23294459131218325787 0.0015469999999983968797 rpy=3.4553794287655741425e-15 -1.8631702197740713788e-17 3.141592653589793116, axis 0 0 1, limit effort=8 velocity=12
- added joint right_knee_motor_to_thigh: type fixed, parent right_thigh_link, child right_knee_motor, origin xyz=-3.7073482355150927381e-05 -0.2329445913121831746 -0.0015469999999983968797 rpy=-3.1415926535897900074 2.1655023358986328438e-17 3.141592653589793116, axis 0 0 1, limit effort=8 velocity=12
- joint left_ankle_joint: child left_foot -> left_foot_10_dof_link; limit lower=-0.52359877559829881566 upper=0.52359877559829881566 effort=8 velocity=7 -> lower=-0.69813170079773179122 upper=0.69813170079773179122 effort=8 velocity=12; origin xyz=-0.0032963899599866147705 -0.2668032164997911071 -0.012956114963095899384 rpy=-3.1415926535897926719 -2.7216398458847901519e-16 -7.5454898815966969652e-11 -> xyz=3.2816069426878924364e-06 -0.033999999841633266051 0.0040000000000006558087 rpy=3.1415926535897900074 -2.7014812817776049377e-17 1.6276071021687969344e-21; parent left_shin -> left_ankle_motor
- joint left_hip_pitch_joint: child left_thigh_assembled_link -> left_thigh_link; limit lower=-1.570796326794896558 upper=0.34906585039886589561 effort=8 velocity=7 -> lower=-1.570796326794896558 upper=0.34906585039886589561 effort=8 velocity=12; origin xyz=-0.02071448272095952059 1.2195219323135608747e-06 0.056302758297119837039 rpy=1.8014407889166555456e-05 -1.570796276518905854 0 -> xyz=-0.020714482720959687123 1.219521932285805299e-06 0.056302758297119850917 rpy=1.8014407889166545292e-05 -1.5707963265881343951 0
- joint left_hip_roll_joint: limit lower=-0.34906585039886589561 upper=0.34906585039886589561 effort=8 velocity=7 -> lower=-0.34906585039886589561 upper=0.34906585039886589561 effort=8 velocity=12; origin xyz=-0.020714482720959499773 1.219521932285805299e-06 0.056302758297119864794 rpy=1.5707963267949003328 -6.9790457465458354129e-11 1.5708143412027857355 -> xyz=-0.020714482720959506712 1.2195219322996830869e-06 0.056302758297119871733 rpy=1.5707963267949003328 -6.9790457465458354129e-11 1.5708143412027857355
- joint left_hip_yaw_joint: limit lower=-0.34906585039886589561 upper=0.34906585039886589561 effort=8 velocity=7 -> lower=-0.34906585039886589561 upper=0.34906585039886589561 effort=8 velocity=12; origin xyz=-0.015448260793301492322 0.090058795475540909248 -0.040999998961279135457 rpy=3.1415926535190985547 -5.0144678432644649869e-08 0.0027836016256884551709 -> xyz=-0.015448260799158839915 0.090058795475540923126 -0.040999998961279135457 rpy=3.1415926535190985547 -5.0144678432644649869e-08 0.0027836016256884551709
- joint left_knee_joint: child left_shin -> left_shin_motor_down_link; limit lower=-0.87266462599716476678 upper=-0 effort=8 velocity=7 -> lower=-0.69813170079773179122 upper=-0 effort=8 velocity=12; origin xyz=-1.1791795445983965784e-05 0.26696937369610784785 -0.0055469999999987473771 rpy=-3.141592653589793116 1.3506088249452880441e-15 -1.5226585619511279746e-21 -> xyz=3.2816069428370786554e-06 -0.033999999841633321562 0.0040000000000005586642 rpy=-4.8921743121386886771e-15 -7.4991735506070378833e-18 -5.0069228532984672229e-08; parent left_thigh_assembled_link -> left_knee_motor
- joint right_ankle_joint: child right_foot -> right_foot_10_dof_link; limit lower=-0.52359877559829881566 upper=0.52359877559829881566 effort=8 velocity=7 -> lower=-0.69813170079773179122 upper=0.69813170079773179122 effort=8 velocity=12; origin xyz=0.003347892444654266414 0.26680257520792799442 -0.012956114963096218573 rpy=3.141592653589793116 2.7929081732228866844e-16 -1.0807875709168855358e-18 -> xyz=3.2816069426878924364e-06 -0.033999999841633155029 0.0040000000000004060086 rpy=-3.1415926535897900074 2.1720554068008287129e-18 -3.141592653589793116; parent right_shin -> right_ankle_motor
- joint right_hip_pitch_joint: child right_thigh_assembled_link -> right_thigh_link; limit lower=-0.34906585039886589561 upper=1.570796326794896558 effort=8 velocity=7 -> lower=-0.34906585039886589561 upper=1.570796326794896558 effort=8 velocity=12; origin xyz=0.020714482720954302541 -1.2192523383830478068e-06 0.056297241554987505208 rpy=-3.1415746391817331862 -1.5707962265083690312 0 -> xyz=0.020714482720954302541 -1.219252338369170019e-06 0.056297241554987505208 rpy=-3.1415746391817331862 -1.5707963267916837946 0
- joint right_hip_roll_joint: limit lower=-0.34906585039886589561 upper=0.34906585039886589561 effort=8 velocity=7 -> lower=-0.34906585039886589561 upper=0.34906585039886589561 effort=8 velocity=12; origin xyz=0.020714482720954306011 -1.219252338369170019e-06 0.056297241554987532963 rpy=1.57079632679489678 3.2127874593201277269e-12 -1.5707783123868368502 -> xyz=0.02071448272095430948 -1.219252338369170019e-06 0.056297241554987512147 rpy=1.57079632679489678 3.2127874593201277269e-12 -1.5707783123868368502
- joint right_hip_yaw_joint: limit lower=-0.34906585039886589561 upper=0.34906585039886589561 effort=8 velocity=7 -> lower=-0.34906585039886589561 upper=0.34906585039886589561 effort=8 velocity=12; origin xyz=-0.015446141467287999999 -0.089944678857579729581 -0.040999998973574106054 rpy=3.1415926535209051096 5.0144680946418486686e-08 3.141592653589793116 -> xyz=-0.015446141460225827971 -0.089944678857579563047 -0.040999998973574099115 rpy=3.1415926535209051096 5.0144680946418486686e-08 3.141592653589793116
- joint right_knee_joint: child right_shin -> right_shin_motor_down_link; limit lower=-0 upper=0.87266462599716476678 effort=8 velocity=7 -> lower=-0 upper=0.69813170079773179122 effort=8 velocity=12; origin xyz=6.3326415581054645854e-05 -0.26696936644585766985 -0.0055469999999988722772 rpy=-3.141592653589793116 -2.0800098087738670828e-17 6.9476554009553828245e-20 -> xyz=-3.2816069417858362289e-06 -0.033999999841633099518 0.0039999999999996982414 rpy=3.4474478122475132731e-15 6.7955268797642522473e-20 -3.1415925533000530478; parent right_thigh_assembled_link -> right_knee_motor
- joint weight_to_base: limit effort=8 velocity=7 -> effort=8 velocity=12; origin xyz=0.021893045761037083913 6.424156877995459633e-05 0.60300000290498989575 rpy=-3.1415926535209051096 -5.0144680946549981934e-08 -1.4608935690811071798e-18 -> xyz=0.031893040747171287619 6.4241565289009446731e-05 0.70300000340643686858 rpy=-3.1415926535209051096 -5.0144680395463669448e-08 7.1773723064297755686e-11
